Commit message: UPDATED JUMPING AMCL with fixed TF! Added Spin Code for Wheel Seperation Calibration.

File: src/ui_ws/urdf/gazebo_control.xacro (robot description, xacro)
@@ -6,5 +6,5 @@
             <left_joint>left_wheel_joint</left_joint>
             <right_joint>right_wheel_joint</right_joint>
-            <wheel_separation>0.51</wheel_separation>
+            <wheel_separation>0.525</wheel_separation>
             <wheel_diameter>0.2</wheel_diameter>
             <!-- Limits -->

File: src/ui_ws/urdf/robot_core.xacro (robot description, xacro)
@@ -10,5 +10,5 @@
     <xacro:property name="wheel_mass" value="1.5"/>
     <xacro:property name="wheel_offset_x" value="0.40"/>
-    <xacro:property name="wheel_offset_y" value="0.255"/>
+    <xacro:property name="wheel_offset_y" value="0.2475"/>
     <xacro:property name="caster_wheel_radius" value="0.038"/>
     <xacro:property name="caster_wheel_mass" value="0.4"/>
