Commit message: feat: integrate reflector localization and overhaul core mission managers
- Implement new 'next_ros2ws_reflector' package for high-precision localizer using map-odom broadcasting
- Overhaul 'zone_manager' and 'map_layer_manager' with extended functionality and robust state handling
- Enhance 'db_manager' and 'ros_bridge' to support expanded mission metadata and real-time telemetry
- Improve 'shelf_detector' with optimized geometric refinement and automated unit tests
- Standardize robot profiles (ugv-01/02) and synchronize navigation parameters
- Refactor project documentation (AGENTS.md) and remove legacy TODO files
- Clean up workspace by migrating deprecated scripts to 'unused_script/'

File: src/ui_ws/config/robot_profiles/artifacts/ugv-01/v7/compiled.urdf (robot description, URDF)
Before this commit: robot UGV_01, 12 links, 11 joints
Joints:
- removed joint base_link_to_base_footprint
- added joint base_footprint_to_base_link: type fixed, parent base_footprint, child base_link, origin xyz=0.000000 0.000000 0.000000 rpy=0.000000 0.000000 0.000000
- joint base_link_to_left_wheel: origin xyz=0.000000 0.255000 0.000000 rpy=-1.570796 0.000000 0.000000 -> xyz=0.000000 0.247500 0.000000 rpy=-1.570796 0.000000 0.000000
- joint base_link_to_right_wheel: origin xyz=0.000000 -0.255000 0.000000 rpy=1.570796 0.000000 0.000000 -> xyz=0.000000 -0.247500 0.000000 rpy=1.570796 0.000000 0.000000
